File: Src/First_Distortion_FD-1.sch (KiCad schematic (older format))
At the start: 36 parts, among them X1 DC_Jack_PCB, X2 DC_Jack_Wire, X3 Battery_Conn, X4 CON

Commit message: Оформление рамки схемы
Other:
- note removed: "Схема электрическая принципиальная"
Changed lines of the file:
@@
 EESchema Schematic File Version 4
-LIBS:First_Distortion_FD-1-cache
-EELAYER 26 0
+EELAYER 30 0
 EELAYER END
 $Descr A4 8268 11693 portrait
 encoding utf-8
 Sheet 1 1
-Title "First Distortion FD-1"
+Title "Эффект гитарный\\nFirst Distortion FD-1\\nСхема электрическая\\nпринципиальная"
 Date "11.21"
 Rev "0"
-Comp "Litone Electronics"
-Comment1 ""
-Comment2 ""
+Comp "Litone Lab"
+Comment1 "2026080016.001 Э3"
+Comment2 "Алимов"
 Comment3 ""
-Comment4 "Алимов"
+Comment4 ""
 $EndDescr
 $Comp
@@
 Text Notes 4400 3100 0    59   ~ 0
 "SIM/ASIM"\n\n
-Text Notes 3400 10850 0    87   ~ 0
-Схема электрическая принципиальная
 $Comp
 L Switch:SW_SPST S2

Commit message: Первая итерация формирования BOM, 3D модели
Parts:
- C1, C9: IPN (none) -> C_THT_RECT-L7-W2.5-H6.5_1n; MPN (none) -> B32529C0102; Manufacturer (none) -> Epcos; Name (none) -> Конденсатор THT MKT 1 нФ ±20%, 63 В, ДхШхВ 7х2,5х6,5 мм, ша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
- C2: IPN (none) -> C_THT_RECT-L7-W2.5-H6.5_10n; MPN (none) -> B32529C0103; Manufacturer (none) -> Epcos; Name (none) -> Конденсатор THT MKT 10 нФ ±20%, 63 В, ДхШхВ 7х2,5х6,5 мм, ш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
- C3: IPN (none) -> C_THT_RECT-L7-W2.5-H6.5_47n; MPN (none) -> B32529C0473; Manufacturer (none) -> Epcos; Name (none) -> Конденсатор THT MKT 47 нФ ±20%, 63 В, ДхШхВ 7х2,5х6,5 мм, ш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
- C4: IPN (none) -> C_THT_RAD-D5-H11_100u; MPN (none) -> JRB1C101M02000500110; Manufacturer (none) -> JB; Name (none) -> Конденсатор THT электролитич. алюм. радиальный 100 мкФ ±20%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
- C5: IPN (none) -> C_THT_RECT-L5-W2.5-H5_10p; MPN (none) -> JYM1H100JBN; Manufacturer (none) -> JB; Name (none) -> Конденсатор THT MLCC NP0 дисковый 10 пФ ±5%, 50 В, ØхШ 5х2,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
- C6, C7: IPN (none) -> C_THT_RAD-D5-H11_1u; MPN (none) -> JRB1H010M02000500110; Manufacturer (none) -> JB; Name (none) -> Конденсатор THT электролитич. алюм. радиальный 1 мкФ ±20%, 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
- C8: IPN (none) -> C_THT_RECT-L5-W2.5-H5_100n; Name (none) -> Конденсатор THT X5R дисковый 100 нФ ±20%, 50 В, ØхШ 5х2,5 м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
- DA1: IPN (none) -> D_THT_DIP-8_uA741; Name (none) -> Микросхема uA741, DIP-8
- HL1: IPN (none) -> LED_THT_D3_Red; Name (none) -> Светодиод выводной красный, Ø 3 мм
- R1, R5, R6, R7, R8: IPN (none) -> R_THT_DIN0207_1M; Name (none) -> Резистор THT металлоплёночный DIN0207 1 МОм ±5%, 0,25 Вт
- R10, R4: IPN (none) -> R_THT_DIN0207_10k; Name (none) -> Резистор THT металлоплёночный DIN0207 10 кОм ±5%, 0,25 Вт
- R11: IPN (none) -> R_SMD_0805_0R; Name (none) -> Резистор SMD 0805 0 Ом
- R2, R9: IPN (none) -> R_THT_DIN0207_4k7; Name (none) -> Резистор THT металлоплёночный DIN0207 4,7 кОм ±5%, 0,25 Вт
- R3: IPN (none) -> R_THT_DIN0207_10R; Name (none) -> Резистор THT металлоплёночный DIN0207 10 Ом ±5%, 0,25 Вт
- RP1: Alt1_IPN (none) -> RP_THT_RV16AF-20_C500k; Alt1_Name (none) -> Потенциометр RV16AF-20 500 кОм, RevLog (C); IPN (none) -> RP_THT_RV16AF-10_C500k; Name (none) -> Потенциометр RV16AF-10 500 кОм, RevLog (C)
- RP2: Alt1_IPN (none) -> RP_THT_RV16AF-20_A50k; Alt1_Name (none) -> Потенциометр RV16AF-20 50 кОм, Log (A); IPN (none) -> RP_THT_RV16AF-10_A50k; Name (none) -> Потенциометр RV16AF-10 50 кОм, Log (A)
- S1: Alt1_IPN (none) -> S_THT_SF17020F-0302_3PDT; Alt1_Name (none) -> Переключатель ножной 3PDT SF17020F-0302; IPN (none) -> S_THT_SF17010F-0302_3PDT; Name (none) -> Переключатель ножной 3PDT SF17010F-0302
- S2: IPN (none) -> S_THT_SMTS-101; Name (none) -> Микротумблер SMTS-101, ON-OFF, SPST, установочное отверстие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
- VD1: value 1N4007 -> 1N4001; IPN (none) -> VD_THT_DO-41_1N4001; Name (none) -> Диод 1N4001 (DO-41); Note (none) -> Любой диод DO-41 средней мощности, V > 25 В
- VD2, VD3, VD4: IPN (none) -> VD_THT_DO-35_1N34; Name (none) -> Диод германиевый 1N34; Note (none) -> Любой выводной германиевый маломощный диод (макс. размер DO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
- X1: IPN (none) -> X_THT_DS-210B-2.1x5.5; Name (none) -> Гнездо DS-210B, 2,1х5,5 мм, пайка на плату
- X2: IPN (none) -> X_THT_XS-2.1x5.5-Panel-D11; Name (none) -> Гнездо питания 2,1х5,5 мм, на панель, крепёжное отверстие Ø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
- X3: IPN (none) -> X_9V-Bat-Snap; Name (none) -> Разъём для батареи типа \"Крона\" боковой
- XS1, XS2: IPN (none) -> X_THT_NMJ6HCD2; Name (none) -> Гнездо Jack 6,3 мм NMJ6HCD2, TRS
