File: Src/First_Distortion_FD-1.kicad_pcb (KiCad board)
At the start: 2 copper layers, 54 x 73.5 mm, 40 parts, among them X1 DC_Jack_PCB, X2 DC_Jack_Wire, X3 Battery_Conn, X4 CON

Commit message: Переход на KiCAD 10, формирование вариантов
* Запустил проект в KiCAD 10
* Добавил варианты исполнения
Other:
- net class Default removed
