File: Src/First_Distortion_FD-1.kicad_pcb (KiCad board)
At the start: 2 copper layers, 54 x 73.5 mm, 40 parts, among them X1 DC_Jack_PCB, X2 DC_Jack_Wire, X3 Battery_Conn, X4 CON

Commit message: Подготовка черновика СБ
Parts:
- DA1: value MAA741 -> uA741
- HL1: value 3mm red -> RED
- S1: value 3PDT -> SF17010F-0302
- S2: value SW_SPST -> MTS-101
- VD1: value 1N4007 -> 1N4001
- VD2, VD3, VD4: value 1N34 -> 1N34A
- X1: value DC_Jack_PCB -> KLS1-DC-005A-2.0
- X2: value DC_Jack_Wire -> KLS1-DC-022B-2.0
- X3: value Battery_Conn -> ~
- X4: value CON -> ~
- XS1, XS2: value Jack_6.3 -> NMJ6HCD2
- moved ? 30.5 mm to (128.8, 54.5)
- moved C1 30.5 mm to (128.2, 111.5)
- moved C2 30.5 mm to (135.2, 84.0)
- moved C3 30.5 mm to (109.2, 80.5)
- moved C4 30.5 mm to (120.8, 71.5)
- moved C5 30.5 mm to (99.8, 64.0)
- moved C6 30.5 mm to (133.8, 79.5)
- moved C7 30.5 mm to (96.2, 66.5)
- moved C8 30.5 mm to (117.2, 68.5)
- moved C9 30.5 mm to (122.8, 84.0)
- moved DA1 30.5 mm to (106.8, 76.5)
- moved G*** 30.5 mm to (132.8, 118.5)
- moved G*** 30.5 mm to (92.2, 57.0)
- moved R1 30.5 mm to (126.6, 108.0)
- moved R10 30.5 mm to (103.8, 77.0)
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Connections:
- net GND renamed GND_AAV
- DA1 pad 1: Net-(DA1-Pad1) -> unconnected-(DA1A-NC-Pad1)
- DA1 pad 5: Net-(DA1-Pad5) -> unconnected-(DA1A-NC-Pad5)
- S1 pad 6: Net-(S1-Pad6) -> unconnected-(S1-Pad6)
- XS1 pad 5: Net-(XS1-Pad5) -> unconnected-(XS1-Pad5)
Other:
- board text added: "1 К контактной площадке Х4 паять провод поз.25 длиной 50 мм. Ко второму концу провода паять лепесток поз.26. Концы проводов предварительно зачистить и залудить 2 К потенциометрам RP1, RP2 паять разъёмы поз.27, как показано на чертеже. Из разъёмов предварительно удалить контакты 2 и 4 3 К контактам 1 и 2 переключателя S2 паять провод поз.25 длиной по 50 мм. Вторые концы проводов паять к соответств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"
- board text added: "Сторона компонентов"
- board text added: "Сторона пайки"
- board text removed: "Развёртка корпуса"

Commit message: Начало работы над СБ, дополнение ExtraBOM (SW-PAN)
Other:
- board text added: "1 К контактной площадке Х4 паять провод МГШВ-0,2 кв.мм (AWG24) черный поз.? длиной 50 мм. Ко второму концу провода паять лепесток 1-2-13-36 поз.?. Концы проводов предварительно зачистить и залудить 2 К потенциометрам RP1, RP2 паять разъёмы PLH-5 поз.?, как показано на чертеже. Из разъёмов предварительно удалить контакты 2 и 4 3 К контактам 1 и 2 переключателя S2 паять провод МГШВ-0,2 кв.мм (AWG24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"
- board text removed: "0"
- board text removed: "1 К контактной площадке Х4 паять провод поз.25 длиной 50 мм. Ко второму концу провода паять лепесток поз.26. Концы проводов предварительно зачистить и залудить 2 К потенциометрам RP1, RP2 паять разъёмы поз.27, как показано на чертеже. Из разъёмов предварительно удалить контакты 2 и 4 3 К контактам 1 и 2 переключателя S2 паять провод поз.25 длиной по 50 мм. Вторые концы проводов паять к соответств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"
