File: Src/First_Distortion_FD-1.kicad_sch (KiCad schematic)
At the start: 36 parts, among them X1 DC_Jack_PCB, X2 DC_Jack_Wire, X3 Battery_Conn, X4 CON

Commit message: pcba: Предварительное приведение в порядок BOM
Parts:
- C1, C9: IPN C_THT_RECT-L7-W2.5-H6.5_1n -> (none); Material (none) -> MKT; Name Конденсатор THT MKT 1 нФ ±20%, 63 В, ДхШхВ 7х2,5х6,5 мм, ша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 -> Конденсатор THT металлоплёночный; Package (none) -> C-THT-RECT-L7-W2.5-H6.5; PinPitch (none) -> 5; Tolerance (none) -> 20%; Voltage (none) -> 63V
- C2: IPN C_THT_RECT-L7-W2.5-H6.5_10n -> (none); Material (none) -> MKT; Name Конденсатор THT MKT 10 нФ ±20%, 63 В, ДхШхВ 7х2,5х6,5 мм, ш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 -> Конденсатор THT металлоплёночный; Package (none) -> C-THT-RECT-L7-W2.5-H6.5; PinPitch (none) -> 5; Tolerance (none) -> 20%; Voltage (none) -> 63V
- C3: IPN C_THT_RECT-L7-W2.5-H6.5_47n -> (none); Material (none) -> MKT; Name Конденсатор THT MKT 47 нФ ±20%, 63 В, ДхШхВ 7х2,5х6,5 мм, ш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 -> Конденсатор THT металлоплёночный; Package (none) -> C-THT-RECT-L7-W2.5-H6.5; PinPitch (none) -> 5; Tolerance (none) -> 20%; Voltage (none) -> 63V
- C4: IPN C_THT_RAD-D5-H11_100u -> (none); Material (none) -> AL-EL; Name Конденсатор THT электролитич. алюм. радиальный 100 мкФ ±20%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 -> Конденсатор THT электролитический алюминиевый; Package (none) -> C-THT-RADIAL-D5-H11; PinPitch (none) -> 2.5; Temperature (none) -> 85 °C; Tolerance (none) -> 20%; Voltage (none) -> 16V
- C5: IPN C_THT_RECT-L5-W2.5-H5_10p -> (none); Material (none) -> NP0; Name Конденсатор THT MLCC NP0 дисковый 10 пФ ±5%, 50 В, ØхШ 5х2,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 -> Конденсатор THT керамический; Package (none) -> C-THT-RECT-L5-W2.5-H5; PinPitch (none) -> 5; Tolerance (none) -> 5%; Voltage (none) -> 50V
- C6: IPN C_THT_RAD-D5-H11_1u -> (none); Material (none) -> TA-EL; Name Конденсатор THT электролитич. алюм. радиальный 1 мкФ ±20%, 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 -> Конденсатор THT электролитический танталовый; Package (none) -> C-THT-RADIAL-D5-H11; PinPitch (none) -> 2.5; Tolerance (none) -> 10%; Voltage (none) -> 50V
- C7: IPN C_THT_RAD-D5-H11_1u -> (none); Material (none) -> AL-EL; Name Конденсатор THT электролитич. алюм. радиальный 1 мкФ ±20%, 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 -> Конденсатор THT электролитический алюминиевый; Package (none) -> C-THT-RADIAL-D5-H11; PinPitch (none) -> 2.5; Temperature (none) -> 85 °C; Tolerance (none) -> 20%; Voltage (none) -> 50V
- C8: IPN C_THT_RECT-L5-W2.5-H5_100n -> (none); Material (none) -> X5R; Name Конденсатор THT X5R дисковый 100 нФ ±20%, 50 В, ØхШ 5х2,5 м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 -> Конденсатор THT керамический; Package (none) -> C-THT-RECT-L5-W2.5-H5; PinPitch (none) -> 5; Tolerance (none) -> 20%; Voltage (none) -> 50V
- DA1: value MAA741 -> uA741; IPN D_THT_DIP-8_uA741 -> (none); Name Микросхема uA741, DIP-8 -> Микросхема; Package (none) -> DIP8
- HL1: value 3mm red -> RED; IPN LED_THT_D3_Red -> (none); Name Светодиод выводной красный, Ø 3 мм -> Светодиод THT, Ø 3 мм, красный; Package (none) -> LED-THT-D3
- R1, R5, R6, R7, R8: IPN R_THT_DIN0207_1M -> (none); Name Резистор THT металлоплёночный DIN0207 1 МОм ±5%, 0,25 Вт -> Резистор THT металлоплёночный; Package (none) -> DIN0207; Power (none) -> 0.125W; Tolerance (none) -> 5%
- R10, R4: IPN R_THT_DIN0207_10k -> (none); Name Резистор THT металлоплёночный DIN0207 10 кОм ±5%, 0,25 Вт -> Резистор THT металлоплёночный; Package (none) -> DIN0207; Power (none) -> 0.125W; Tolerance (none) -> 5%
- R11: IPN R_SMD_0805_0R -> (none); Name Резистор SMD 0805 0 Ом -> Резистор SMD металлоплёночный; Package (none) -> SMD0805; Power (none) -> 0.125W
- R2, R9: IPN R_THT_DIN0207_4k7 -> (none); Name Резистор THT металлоплёночный DIN0207 4,7 кОм ±5%, 0,25 Вт -> Резистор THT металлоплёночный; Package (none) -> DIN0207; Power (none) -> 0.125W; Tolerance (none) -> 5%
- R3: IPN R_THT_DIN0207_10R -> (none); Name Резистор THT металлоплёночный DIN0207 10 Ом ±5%, 0,25 Вт -> Резистор THT металлоплёночный; Package (none) -> DIN0207; Power (none) -> 0.125W; Tolerance (none) -> 5%
- RP1: IPN RP_THT_RV16AF-10_C500k -> (none); Manufacturer (none) -> Alpha; Name Потенциометр RV16AF-10 500 кОм, RevLog (C) -> Потенциометр RV16AF-10; Package (none) -> RV16AF-10
- RP2: IPN RP_THT_RV16AF-10_A50k -> (none); Manufacturer (none) -> Alpha; Name Потенциометр RV16AF-10 50 кОм, Log (A) -> Потенциометр RV16AF-10; Package (none) -> RV16AF-10
- S1: value 3PDT -> SF17010F-0302; IPN S_THT_SF17010F-0302_3PDT -> (none); Manufacturer (none) -> Alpha; Package (none) -> SF17010F-0302
- S2: value SW_SPST -> MTS-101; IPN S_THT_SMTS-101 -> (none); Name Микротумблер SMTS-101, ON-OFF, SPST, установочное отверстие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 -> Миниатюрный переключатель MTS-101; Package (none) -> MTS-101
- VD1: IPN VD_THT_DO-41_1N4001 -> (none); Material (none) -> Si; Name Диод 1N4001 (DO-41) -> Диод кремниевый; Note Любой диод DO-41 средней мощности, V > 25 В -> (none); Package (none) -> DO-41; Voltage (none) -> 25V
- VD2, VD3, VD4: IPN VD_THT_DO-35_1N34 -> (none); Material (none) -> Ge; Name Диод германиевый 1N34 -> Диод германиевый; Note Любой выводной германиевый маломощный диод (макс. размер DO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 -> (none); Package (none) -> DO-35
- X1: value DC_Jack_PCB -> KLS1-DC-005A-2.0; IPN X_THT_DS-210B-2.1x5.5 -> (none); MPN (none) -> KLS1-DC-005A-2.0; Manufacturer (none) -> KLS; Name Гнездо DS-210B, 2,1х5,5 мм, пайка на плату -> Гнездо питания KLS1-DC-005A-2.0; Package (none) -> KLS1-DC-005A-2.0
- X2: value DC_Jack_Wire -> KLS1-DC-022B-2.0; IPN X_THT_XS-2.1x5.5-Panel-D11 -> (none); MPN (none) -> KLS1-DC-022B-2.0; Manufacturer (none) -> KLS; Name Гнездо питания 2,1х5,5 мм, на панель, крепёжное отверстие Ø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 -> Гнездо питания KLS1-DC-022B-2.0; Package (none) -> KLS1-DC-022B-2.0
- X3: value Battery_Conn -> (none); IPN X_9V-Bat-Snap -> (none); Name Разъём для батареи типа "Крона" боковой -> Разъём для батареи типа "Крона" боковой
- X4: value CON -> (none)
- XS1, XS2: value Jack_6.3 -> NMJ6HCD2; IPN X_THT_NMJ6HCD2 -> (none); MPN (none) -> NMJ6HCD2; Manufacturer (none) -> Neutrik; Name Гнездо Jack 6,3 мм NMJ6HCD2, TRS -> Гнездо Jack 6,3 мм TRS NMJ6HCD2
Other:
- company: Litone Lab -> (none)
- title: Эффект гитарный\nFirst Distortion FD-1\nСхема электрическая\nпринципиальная -> Эффект дисторшн\nFD-1\nСхема электрическая\nпринципиальная

Commit message: Продолжение наполнения BOM для разных исполнений
Parts:
- C1, C9: Chipdip_link (none) -> https://www.chipdip.ru/product/b32529c0102j000-0.001-mkf-40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; Diy-tubes_alt_link (none) -> https://diy-tubes.ru/index.php?route=product/product&path=2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; Diy-tubes_link (none) -> https://diy-tubes.ru/index.php?route=product/product&path=2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
- C2: Chipdip_link (none) -> https://www.chipdip.ru/product/b32529c0103j000-tdk-80083940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; Diy-tubes_alt_link (none) -> https://diy-tubes.ru/index.php?route=product/product&path=2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; Diy-tubes_link (none) -> https://diy-tubes.ru/index.php?route=product/product&path=2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
- C3: Chipdip_link (none) -> https://www.chipdip.ru/product/mkt-film-capacitor-47-nf-10-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; Diy-tubes_alt_link (none) -> https://diy-tubes.ru/index.php?route=product/product&path=2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; Diy-tubes_link (none) -> https://diy-tubes.ru/index.php?route=product/product&path=2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
- C4: Chipdip_link (none) -> https://www.chipdip.ru/product/100mkf-16v-105-c-20-5x11mm-p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
- C5: Chipdip_link (none) -> https://www.chipdip.ru/product/k10-17b-10pf-npo-5-0805-jym1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; Diy-tubes_alt_link (none) -> https://diy-tubes.ru/index.php?route=product/product&path=2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
- C6: Chipdip_link (none) -> https://www.chipdip.ru/product/tc-1-50-kondensator-tantalov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; MPN JRB1H010M02000500110 -> TC-1/50; Manufacturer JB -> SR Passives
- C7: Chipdip_link (none) -> https://www.chipdip.ru/product/1mkf-50v-105-c-20-5x11mm-p-2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; Diy-tubes_alt_link (none) -> https://diy-tubes.ru/index.php?route=product/product&path=2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
- C8: Chipdip_link (none) -> https://www.chipdip.ru/product/k10-17b-1000pf-x7r-10-0805-j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; Diy-tubes_alt_link (none) -> https://diy-tubes.ru/index.php?route=product/product&path=2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; MPN (none) -> JYM1H102KBX; Manufacturer (none) -> JB; Material X5R -> X7R
- DA1: Chipdip_link (none) -> https://www.chipdip.ru/product/ua741cp-universalnyy-odnokan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; Diy-tubes_alt_link (none) -> https://diy-tubes.ru/index.php?route=product/product&path=2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; MPN (none) -> UA741CP; Manufacturer (none) -> TI; Name Микросхема -> Микросхема uA741
- HL1: Chipdip_link (none) -> https://www.chipdip.ru/product/gnl-3012hd-svetodiod-krasnyy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; Diy-tubes_alt_link (none) -> https://diy-tubes.ru/index.php?route=product/product&path=2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; MPN (none) -> GNL-3012HD; Manufacturer (none) -> G-NOR
- R1, R5, R6, R7, R8: Chipdip_link (none) -> https://www.chipdip.ru/product/mfr-25ftf52-1m-0.25vt-1mom-1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; Diy-tubes_alt_link (none) -> https://diy-tubes.ru/index.php?route=product/product&path=2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
- R10, R4: Chipdip_link (none) -> https://www.chipdip.ru/product/mfr-25ftf52-10k-0.25vt-10kom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
- R11: Chipdip_link (none) -> https://www.chipdip.ru/product/cr0805aj-000eas-resa-as-0805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
- R2, R9: Chipdip_link (none) -> https://www.chipdip.ru/product/mf-25-s2-23-0.25vt-4.7-kom-1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; Diy-tubes_alt_link (none) -> https://diy-tubes.ru/index.php?route=product/product&path=2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
- R3: Chipdip_link (none) -> https://www.chipdip.ru/product/mfr-25ftf52-10r-0.25vt-10om-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
- RP1: Alt1_IPN RP_THT_RV16AF-20_C500k -> (none); Alt1_Name Потенциометр RV16AF-20 500 кОм, RevLog (C) -> (none); Diy-tubes_alt_link (none) -> https://diy-tubes.ru/index.php?route=product/product&path=2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; Diy-tubes_link (none) -> https://diy-tubes.ru/index.php?route=product/product&path=2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; MPN (none) -> RV16AF-10-15K-C500k
- RP2: Alt1_IPN RP_THT_RV16AF-20_A50k -> (none); Alt1_Name Потенциометр RV16AF-20 50 кОм, Log (A) -> (none); Diy-tubes_alt_link (none) -> https://diy-tubes.ru/index.php?route=product/product&path=2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; Diy-tubes_link (none) -> https://diy-tubes.ru/index.php?route=product/product&path=2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; MPN (none) -> RV16AF-10-15K-A50k
- S1: Alt1_IPN S_THT_SF17020F-0302_3PDT -> (none); Alt1_Name Переключатель ножной 3PDT SF17020F-0302 -> (none); Diy-tubes_alt_link (none) -> https://diy-tubes.ru/index.php?route=product/product&path=2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; MPN (none) -> SF17010F-0302
- S2: Chipdip_link (none) -> https://www.chipdip.ru/product/mts-101-on-off-mikrotumbler-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; Diy-tubes_alt_link (none) -> https://diy-tubes.ru/index.php?route=product/product&path=2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; Diy-tubes_link (none) -> https://diy-tubes.ru/index.php?route=product/product&path=2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
- VD1: Chipdip_link (none) -> https://www.chipdip.ru/product/1n4001-diod-vypryamitelnyy-1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; Diy-tubes_link (none) -> https://diy-tubes.ru/index.php?route=product/product&path=2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
- VD2, VD3, VD4: value 1N34 -> 1N34A; Chipdip_link (none) -> https://www.chipdip.ru/product/d9b-diod-vypryamitelnyy-malo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; Diy-tubes_link (none) -> https://diy-tubes.ru/index.php?route=product/product&path=2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
- X1: Chipdip_link (none) -> https://www.chipdip.ru/product/kls1-dc-005a-2.0-gnezdo-pita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
- X2, X3: Diy-tubes_link (none) -> https://diy-tubes.ru/index.php?route=product/product&path=2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
- XS1, XS2: Diy-tubes_alt_link (none) -> https://diy-tubes.ru/index.php?route=product/product&path=2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; Diy-tubes_link (none) -> https://diy-tubes.ru/index.php?route=product/product&path=2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

Commit message: Вывод BOM и перечня элементов для всех вариантов
* _EBOM.csv - спецификация, сгенерированная KiCAD
* _PE3.csv - перечень элементов (все элементы по порядку,
без группировки), сгенерированный KiCAD
* _MBOM.csv - производственная спецификация
(EBOM + доп. детали и материалы для сборки платы)
Parts:
- RP1, RP2: Name Потенциометр RV16AF-10 -> Потенциометр RV16AF-10-15K
- VD1: Name Диод кремниевый -> Диод кремниевый 1N4001
- VD2, VD3, VD4: Name Диод германиевый -> Диод германиевый 1N34A
Other:
- title: Эффект дисторшн\nFD-1\nСхема электрическая\nпринципиальная -> Плата эффекта\nдисторшн FD-1\nСхема электрическая\nпринципиальная
Changed lines of the file:
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@@
 	(paper "A4" portrait)
 	(title_block
-		(title "Эффект дисторшн\\nFD-1\\nСхема электрическая\\nпринципиальная")
+		(title "Плата эффекта\\nдисторшн FD-1\\nСхема электрическая\\nпринципиальная")
 		(date "11.21")
 		(rev "0")
@@
 			)
 		)
-		(property "Description" "Любой аналог: КР140УД7, К140УД7, MAA741 и т.д. Можно в металлическом круглом корпусе"
+		(property "Description" "Любой аналог: КР140УД7, К140УД7, MAA741 и т.д. Можно в металлическом круглом корпусе TO-99-8"
 			(at 82.55 62.23 0)
 			(hide yes)
@@
 			)
 		)
-		(property "Description" "Любой аналог: КР140УД7, К140УД7, MAA741 и т.д. Можно в металлическом круглом корпусе"
+		(property "Description" "Любой аналог: КР140УД7, К140УД7, MAA741 и т.д. Можно в металлическом круглом корпусе TO-99-8"
 			(at 123.19 148.59 0)
 			(hide yes)
@@
 			)
 		)
-		(property "Name" "Потенциометр RV16AF-10"
+		(property "Name" "Потенциометр RV16AF-10-15K"
 			(at 68.58 92.71 0)
 			(hide yes)
@@
 			)
 		)
-		(property "Name" "Потенциометр RV16AF-10"
+		(property "Name" "Потенциометр RV16AF-10-15K"
 			(at 165.1 68.58 0)
 			(hide yes)
@@
 			)
 		)
-		(property "Description" "Любой выводной германиевый маломощный диод (макс. размер DO-41)"
+		(property "Description" "Любой германиевый маломощный диод (макс. размер DO-41): Д9, Д310 и т.д."
 			(at 129.54 71.12 0)
 			(hide yes)
@@
 			)
 		)
-		(property "Name" "Диод германиевый"
+		(property "Name" "Диод германиевый 1N34A"
 			(at 129.54 71.12 0)
 			(hide yes)
@@
 			)
 		)
-		(property "Description" "Любой выводной германиевый маломощный диод (макс. размер DO-41)"
+		(property "Description" "Любой германиевый маломощный диод (макс. размер DO-41): Д9, Д310 и т.д."
 			(at 138.43 71.12 0)
 			(hide yes)
@@
 			)
 		)
-		(property "Name" "Диод германиевый"
+		(property "Name" "Диод германиевый 1N34A"
 			(at 138.43 71.12 0)
 			(hide yes)
@@
 			)
 		)
-		(property "Name" "Диод кремниевый"
+		(property "Name" "Диод кремниевый 1N4001"
 			(at 76.2 144.78 0)
 			(hide yes)
@@
 			)
 		)
-		(property "Description" "Любой выводной германиевый маломощный диод (макс. размер DO-41)"
+		(property "Description" "Любой германиевый маломощный диод (макс. размер DO-41): Д9, Д310 и т.д."
 			(at 138.43 82.55 0)
 			(hide yes)
@@
 			)
 		)
-		(property "Name" "Диод германиевый"
+		(property "Name" "Диод германиевый 1N34A"
 			(at 138.43 82.55 0)
 			(hide yes)
