File: Src/First_Distortion_FD-1.kicad_sch (KiCad schematic)
At the start: 36 parts, among them X1 KLS1-DC-005A-2.0, X2 KLS1-DC-022B-2.0

Commit message: Исправление BOM и вывода схемы
* Поправил логику работы с BOM
* Исправил содержимое BOM
* Изменил рамку схемы на стандартную
* Добавил необходимое описание для рамки схемы
Parts:
- R1, R5, R6, R7, R8: MPN (none) -> KLS6-MF-1/4W-1MR-J; Manufacturer (none) -> KLS
- R10, R4: MPN (none) -> KLS6-MF-1/4W-10KR-J; Manufacturer (none) -> KLS
- R11: Chipdip_link https://www.chipdip.ru/product/cr0805aj-000eas-resa-as-0805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 -> https://www.chipdip.ru/product/cr-05fl7-0r-rezistor-tolstop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; MPN (none) -> CR-05JL7----0R; Manufacturer (none) -> VIKING
- R2, R9: MPN (none) -> KLS6-MF-1/4W-4K7R-J; Manufacturer (none) -> KLS
- R3: MPN (none) -> KLS6-MF-1/4W-10R-J; Manufacturer (none) -> KLS
- S2: MPN (none) -> MTS-101; Manufacturer (none) -> RUICHI
- VD1: MPN (none) -> 1N4001; Manufacturer (none) -> DC Components
- VD2, VD3, VD4: value 1N34A -> 1N34A (Д9); MPN (none) -> Д9; Name Диод германиевый 1N34A -> Диод германиевый 1N34A (Д9)
Other:
- company: (none) -> Alimach
- title: Плата эффекта\nдисторшн FD-1\nСхема электрическая\nпринципиальная -> Эффект дисторшн FD-1. Схема электрич. принципиальная
- moved on the sheet: C1, C2, C3, C4, C5, C6, C7, C8, C9, DA1A, DA1B, HL1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
